File: KiCAD/prototype/prototype.sch (KiCad schematic (older format))
At the start: 2 parts

Commit message: Revert "Merge branch 'devel' into luis"
This reverts commit 12b203dde500fe9434468d0bdc425e41ba632681, reversing
changes made to 5ff5ea5b06c891ff9ca50429f18fec54b7dc7daa.
Connections:
- net labels added: BATTERY
- wire segments 17 -> 23
Changed lines of the file:
@@
-$EndSheet
-$Sheet
-S 2450 2350 650  800
-U 5FAF93BD
-F0 "BatteryCharger" 50
-F1 "BatteryCharger.sch" 50
-F2 "THERM" I L 2450 2900 50
-F3 "ISET" I L 2450 2750 50
-F4 "CE" I L 2450 2600 50
-F5 "PGOOD" I L 2450 2450 50
-F6 "CHG" I R 3100 2750 50
-F7 "OUT" I R 3100 2600 50
-F8 "GND" I R 3100 2450 50
-F9 "VLIPO" I L 2450 3050 50
 $EndSheet
 $Sheet
@@
 Text Label 3350 3850 0    50   ~ 0
 GND
-Text Label 3450 2450 0    50   ~ 0
-GND
-Text Label 3450 2600 0    50   ~ 0
-Vin_Buck
-Wire Wire Line
-	3100 2600 3450 2600
-Wire Wire Line
-	3100 2450 3450 2450
 Wire Wire Line
 	3000 3550 3350 3550
@@
 Text Label 5150 4800 2    50   ~ 0
 Anemometer_Out
+$Sheet
+S 2450 2300 700  600
+U 5FB60B8D
+F0 "Charger" 50
+F1 "Adafruit_BQ24074.sch" 50
+F2 "THERM" I L 2450 2800 50
+F3 "ISET" I L 2450 2700 50
+F4 "CE" I L 2450 2600 50
+F5 "PGOOD" I L 2450 2500 50
+F6 "CHG" I L 2450 2400 50
+F7 "OUT" I R 3150 2400 50
+F8 "VLIPO" I R 3150 2500 50
+F9 "GND" I R 3150 2600 50
+$EndSheet
+Wire Wire Line
+	3150 2400 3500 2400
+Wire Wire Line
+	3150 2500 3500 2500
+Wire Wire Line
+	3150 2600 3500 2600
+Wire Wire Line
+	2450 2400 2150 2400
+Wire Wire Line
+	2450 2500 2150 2500
+Wire Wire Line
+	2450 2600 2150 2600
+Wire Wire Line
+	2450 2700 2150 2700
+Wire Wire Line
+	2450 2800 2150 2800
+Text Label 3500 2400 0    50   ~ 0
+Vin_Buck
+Text Label 3500 2600 0    50   ~ 0
+GND
+Text Label 3500 2500 0    50   ~ 0
+BATTERY
 $EndSCHEMATC
