File: KiCAD/prototype/Anemometer.sch (KiCad schematic (older format))
At the start: 0 parts

Commit message: Improve Anemometer schematics
Parts:
- added J?: RJ22, symbol Connector:RJ22
- added SW?: SW_Reed, symbol Switch:SW_Reed
Connections:
- net Out: now also J?.3, SW?.1
- new net COM: J?.2, SW?.2
Changed lines of the file:
@@
 $Descr A4 11693 8268
 encoding utf-8
-Sheet 6 6
+Sheet 5 6
 Title ""
 Date ""
@@
 Comment4 ""
 $EndDescr
-Text HLabel 5350 3050 0    50   Input ~ 0
-Vin
-Text HLabel 5350 2850 0    50   Input ~ 0
+Text HLabel 5950 4050 3    50   Input ~ 0
+COM
+Text HLabel 5950 3950 1    50   Input ~ 0
 Out
+$Comp
+L Switch:SW_Reed SW?
+U 1 1 5FB811D2
+P 6400 3950
+F 0 "SW?" H 6400 4172 50  0000 C CNN
+F 1 "SW_Reed" H 6400 4081 50  0000 C CNN
+F 2 "" H 6400 3950 50  0001 C CNN
+F 3 "~" H 6400 3950 50  0001 C CNN
+	1    6400 3950
+	1    0    0    -1
+$EndComp
+$Comp
+L Connector:RJ22 J?
+U 1 1 5FB82337
+P 5300 4050
+F 0 "J?" H 5357 4517 50  0000 C CNN
+F 1 "RJ22" H 5357 4426 50  0000 C CNN
+F 2 "" V 5300 4100 50  0001 C CNN
+F 3 "~" V 5300 4100 50  0001 C CNN
+	1    5300 4050
+	1    0    0    -1
+$EndComp
+Wire Wire Line
+	6200 3950 5700 3950
+Wire Wire Line
+	5700 4050 6750 4050
+Wire Wire Line
+	6750 4050 6750 3950
+Wire Wire Line
+	6750 3950 6600 3950
 $EndSCHEMATC
