File: KiCAD/prototype/Adafruit_BQ24074.sch (KiCad schematic (older format))
At the start: 44 parts

Commit message: Improve looks (minor)
Changed lines of the file:
@@
 L Adafruit_BQ24074-rescue:FRAME_A4_ADAFRUIT-Adafruit_BQ24074-eagle-import-Adafruit_BQ24074-rescue #U$?
 U 1 1 BCE09641
-P 1100 7500
-F 0 "#U$?" H 1100 7500 50  0001 C CNN
-F 1 "FRAME_A4_ADAFRUIT" H 1100 7500 50  0001 C CNN
-F 2 "" H 1100 7500 50  0001 C CNN
-F 3 "" H 1100 7500 50  0001 C CNN
-	1    1100 7500
+P 1450 6750
+F 0 "#U$?" H 1450 6750 50  0001 C CNN
+F 1 "FRAME_A4_ADAFRUIT" H 1450 6750 50  0001 C CNN
+F 2 "" H 1450 6750 50  0001 C CNN
+F 3 "" H 1450 6750 50  0001 C CNN
+	1    1450 6750
 	1    0    0    -1
 $EndComp
@@
 L Adafruit_BQ24074-rescue:MOUNTINGHOLE2.5-Adafruit_BQ24074-eagle-import-Adafruit_BQ24074-rescue U$?
 U 1 1 6E1B97F5
-P 10400 6300
-F 0 "U$?" H 10400 6300 50  0001 C CNN
-F 1 "MOUNTINGHOLE2.5" H 10400 6300 50  0001 C CNN
-F 2 "Adafruit_BQ24074:MOUNTINGHOLE_2.5_PLATED" H 10400 6300 50  0001 C CNN
-F 3 "" H 10400 6300 50  0001 C CNN
-	1    10400 6300
+P 10750 5550
+F 0 "U$?" H 10750 5550 50  0001 C CNN
+F 1 "MOUNTINGHOLE2.5" H 10750 5550 50  0001 C CNN
+F 2 "Adafruit_BQ24074:MOUNTINGHOLE_2.5_PLATED" H 10750 5550 50  0001 C CNN
+F 3 "" H 10750 5550 50  0001 C CNN
+	1    10750 5550
 	1    0    0    -1
 $EndComp
@@
 L Adafruit_BQ24074-rescue:MOUNTINGHOLE2.5-Adafruit_BQ24074-eagle-import-Adafruit_BQ24074-rescue U$?
 U 1 1 649D799B
-P 10800 6300
-F 0 "U$?" H 10800 6300 50  0001 C CNN
-F 1 "MOUNTINGHOLE2.5" H 10800 6300 50  0001 C CNN
-F 2 "Adafruit_BQ24074:MOUNTINGHOLE_2.5_PLATED" H 10800 6300 50  0001 C CNN
-F 3 "" H 10800 6300 50  0001 C CNN
-	1    10800 6300
+P 11150 5550
+F 0 "U$?" H 11150 5550 50  0001 C CNN
+F 1 "MOUNTINGHOLE2.5" H 11150 5550 50  0001 C CNN
+F 2 "Adafruit_BQ24074:MOUNTINGHOLE_2.5_PLATED" H 11150 5550 50  0001 C CNN
+F 3 "" H 11150 5550 50  0001 C CNN
+	1    11150 5550
 	1    0    0    -1
 $EndComp
@@
 L Adafruit_BQ24074-rescue:MOUNTINGHOLE2.5-Adafruit_BQ24074-eagle-import-Adafruit_BQ24074-rescue U$?
 U 1 1 ABBF7E6D
-P 10400 6600
-F 0 "U$?" H 10400 6600 50  0001 C CNN
-F 1 "MOUNTINGHOLE2.5" H 10400 6600 50  0001 C CNN
-F 2 "Adafruit_BQ24074:MOUNTINGHOLE_2.5_PLATED" H 10400 6600 50  0001 C CNN
-F 3 "" H 10400 6600 50  0001 C CNN
-	1    10400 6600
+P 10750 5850
+F 0 "U$?" H 10750 5850 50  0001 C CNN
+F 1 "MOUNTINGHOLE2.5" H 10750 5850 50  0001 C CNN
+F 2 "Adafruit_BQ24074:MOUNTINGHOLE_2.5_PLATED" H 10750 5850 50  0001 C CNN
+F 3 "" H 10750 5850 50  0001 C CNN
+	1    10750 5850
 	1    0    0    -1
 $EndComp
@@
 L Adafruit_BQ24074-rescue:MOUNTINGHOLE2.5-Adafruit_BQ24074-eagle-import-Adafruit_BQ24074-rescue U$?
 U 1 1 FCFA34DC
-P 10800 6600
-F 0 "U$?" H 10800 6600 50  0001 C CNN
-F 1 "MOUNTINGHOLE2.5" H 10800 6600 50  0001 C CNN
-F 2 "Adafruit_BQ24074:MOUNTINGHOLE_2.5_PLATED" H 10800 6600 50  0001 C CNN
-F 3 "" H 10800 6600 50  0001 C CNN
-	1    10800 6600
+P 11150 5850
+F 0 "U$?" H 11150 5850 50  0001 C CNN
+F 1 "MOUNTINGHOLE2.5" H 11150 5850 50  0001 C CNN
+F 2 "Adafruit_BQ24074:MOUNTINGHOLE_2.5_PLATED" H 11150 5850 50  0001 C CNN
+F 3 "" H 11150 5850 50  0001 C CNN
+	1    11150 5850
 	1    0    0    -1
 $EndComp
@@
 L Adafruit_BQ24074-rescue:FIDUCIAL_1MM-Adafruit_BQ24074-eagle-import-Adafruit_BQ24074-rescue FID?
 U 1 1 57AF2ED6
-P 11000 6600
-F 0 "FID?" H 11000 6600 50  0001 C CNN
-F 1 "FIDUCIAL_1MM" H 11000 6600 50  0001 C CNN
-F 2 "Adafruit_BQ24074:FIDUCIAL_1MM" H 11000 6600 50  0001 C CNN
-F 3 "" H 11000 6600 50  0001 C CNN
-	1    11000 6600
+P 11350 5850
+F 0 "FID?" H 11350 5850 50  0001 C CNN
+F 1 "FIDUCIAL_1MM" H 11350 5850 50  0001 C CNN
+F 2 "Adafruit_BQ24074:FIDUCIAL_1MM" H 11350 5850 50  0001 C CNN
+F 3 "" H 11350 5850 50  0001 C CNN
+	1    11350 5850
 	1    0    0    -1
 $EndComp
@@
 L Adafruit_BQ24074-rescue:FIDUCIAL_1MM-Adafruit_BQ24074-eagle-import-Adafruit_BQ24074-rescue FID?
 U 1 1 AD69ACBC
-P 11000 6300
-F 0 "FID?" H 11000 6300 50  0001 C CNN
-F 1 "FIDUCIAL_1MM" H 11000 6300 50  0001 C CNN
-F 2 "Adafruit_BQ24074:FIDUCIAL_1MM" H 11000 6300 50  0001 C CNN
-F 3 "" H 11000 6300 50  0001 C CNN
-	1    11000 6300
+P 11350 5550
+F 0 "FID?" H 11350 5550 50  0001 C CNN
+F 1 "FIDUCIAL_1MM" H 11350 5550 50  0001 C CNN
+F 2 "Adafruit_BQ24074:FIDUCIAL_1MM" H 11350 5550 50  0001 C CNN
+F 3 "" H 11350 5550 50  0001 C CNN
+	1    11350 5550
 	1    0    0    -1
 $EndComp
@@
 L Adafruit_BQ24074-rescue:FIDUCIAL_1MM-Adafruit_BQ24074-eagle-import-Adafruit_BQ24074-rescue FID?
 U 1 1 C6D146FB
-P 10600 6300
-F 0 "FID?" H 10600 6300 50  0001 C CNN
-F 1 "FIDUCIAL_1MM" H 10600 6300 50  0001 C CNN
-F 2 "Adafruit_BQ24074:FIDUCIAL_1MM" H 10600 6300 50  0001 C CNN
-F 3 "" H 10600 6300 50  0001 C CNN
-	1    10600 6300
-	1    0    0    -1
-$EndComp
+P 10950 5550
+F 0 "FID?" H 10950 5550 50  0001 C CNN
+F 1 "FIDUCIAL_1MM" H 10950 5550 50  0001 C CNN
+F 2 "Adafruit_BQ24074:FIDUCIAL_1MM" H 10950 5550 50  0001 C CNN
+F 3 "" H 10950 5550 50  0001 C CNN
+	1    10950 5550
+	1    0    0    -1
+$EndComp
