File: KiCAD/prototype/SoundSensor.sch (KiCad schematic (older format))
At the start: 20 parts, among them J2 TWIG_2.0, U1 LM2904DR, U4 SENSOR-MULPS4CX

Commit message: Improve looks (minor)
Connections:
- wire segments 62 -> 63
Other:
- moved on the sheet: C1, C2, C3, C4, C5, C6, J2, MIC1, MIC2, R1, R2, R3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
