File: KiCAD/prototype/ESP32-DevKitC-V4.sch (KiCad schematic (older format))
At the start: 31 parts

Commit message: Remove test label
Changed lines of the file:
@@
 Wire Wire Line
 	6550 2600 6050 2600
-Wire Wire Line
-	6550 2700 6450 2700
 Text Label 6050 900  0    50   ~ 0
 GND
@@
 Wire Wire Line
 	5050 4850 5500 4850
-Text HLabel 6450 3400 0    50   Input ~ 0
-teste1
-Wire Wire Line
-	6450 3400 6450 2700
-Connection ~ 6450 2700
-Wire Wire Line
-	6450 2700 6050 2700
+Wire Wire Line
+	6050 2700 6550 2700
 $EndSCHEMATC
