File: KiCAD/main/Microcontroller.sch (KiCad schematic (older format))
At the start: 10 parts, among them J5 Conn_02x04_Odd_Even, SW1 BOOT, SW2 RESET, U1 ESP32-WROOM-32

Commit message: Clear anotations
Parts:
- renumbered C1 to C?, C5 to C?, C4 to C?, C2 to C?, C3 to C?, J5 to J?, R2 to R?, SW1 to SW?, SW2 to SW?, U1 to U?
Changed lines of the file:
@@
 $EndDescr
 $Comp
-L RF_Module:ESP32-WROOM-32 U1
+L RF_Module:ESP32-WROOM-32 U?
 U 1 1 5F93B762
 P 8200 3700
-F 0 "U1" H 7750 5050 50  0000 C CNN
+F 0 "U?" H 7750 5050 50  0000 C CNN
 F 1 "ESP32-WROOM-32" H 8600 5050 50  0000 C CNN
 F 2 "RF_Module:ESP32-WROOM-32" H 8200 2200 50  0001 C CNN
@@
 $EndComp
 $Comp
-L power:+3V3 #PWR03
+L power:+3V3 #PWR?
 U 1 1 5F9419AA
 P 1100 2650
-F 0 "#PWR03" H 1100 2500 50  0001 C CNN
+F 0 "#PWR?" H 1100 2500 50  0001 C CNN
 F 1 "+3V3" H 1115 2823 50  0000 C CNN
 F 2 "" H 1100 2650 50  0001 C CNN
@@
 $EndComp
 $Comp
-L Device:R R2
+L Device:R R?
 U 1 1 5F94208F
 P 1100 2900
-F 0 "R2" H 1170 2946 50  0000 L CNN
+F 0 "R?" H 1170 2946 50  0000 L CNN
 F 1 "10kR" H 1170 2855 50  0000 L CNN
 F 2 "Resistor_SMD:R_1206_3216Metric" V 1030 2900 50  0001 C CNN
@@
 $EndComp
 $Comp
-L Device:C C1
+L Device:C C?
 U 1 1 5F9429EB
 P 1100 3300
-F 0 "C1" H 1215 3346 50  0000 L CNN
+F 0 "C?" H 1215 3346 50  0000 L CNN
 F 1 "0.1uF" H 1215 3255 50  0000 L CNN
 F 2 "Capacitor_SMD:C_1206_3216Metric" H 1138 3150 50  0001 C CNN
@@
 $EndComp
 $Comp
-L power:GND #PWR04
+L power:GND #PWR?
 U 1 1 5F942C61
 P 1100 3550
-F 0 "#PWR04" H 1100 3300 50  0001 C CNN
+F 0 "#PWR?" H 1100 3300 50  0001 C CNN
 F 1 "GND" H 1105 3377 50  0000 C CNN
 F 2 "" H 1100 3550 50  0001 C CNN
@@
 	1100 2750 1100 2650
 $Comp
-L power:+3V3 #PWR06
+L power:+3V3 #PWR?
 U 1 1 5F943FB0
 P 7350 1600
-F 0 "#PWR06" H 7350 1450 50  0001 C CNN
+F 0 "#PWR?" H 7350 1450 50  0001 C CNN
 F 1 "+3V3" H 7365 1773 50  0000 C CNN
 F 2 "" H 7350 1600 50  0001 C CNN
@@
 $EndComp
 $Comp
-L Device:C C5
+L Device:C C?
 U 1 1 5F9451F0
 P 7800 1850
-F 0 "C5" H 7915 1896 50  0000 L CNN
+F 0 "C?" H 7915 1896 50  0000 L CNN
 F 1 "0.1uF" H 7915 1805 50  0000 L CNN
 F 2 "Capacitor_SMD:C_1206_3216Metric" H 7838 1700 50  0001 C CNN
@@
 $EndComp
 $Comp
-L Device:C C4
+L Device:C C?
 U 1 1 5F946123
 P 7350 1850
-F 0 "C4" H 7465 1896 50  0000 L CNN
+F 0 "C?" H 7465 1896 50  0000 L CNN
 F 1 "22uF" H 7465 1805 50  0000 L CNN
 F 2 "Capacitor_SMD:C_1206_3216Metric" H 7388 1700 50  0001 C CNN
@@
 	7350 2050 7350 2000
 $Comp
-L power:GND #PWR07
+L power:GND #PWR?
 U 1 1 5F947B11
 P 7350 2100
-F 0 "#PWR07" H 7350 1850 50  0001 C CNN
+F 0 "#PWR?" H 7350 1850 50  0001 C CNN
 F 1 "GND" H 7355 1927 50  0000 C CNN
 F 2 "" H 7350 2100 50  0001 C CNN
@@
 	8200 2300 8200 1650
 $Comp
-L power:GND #PWR08
+L power:GND #PWR?
 U 1 1 5F95286C
 P 8200 5300
-F 0 "#PWR08" H 8200 5050 50  0001 C CNN
+F 0 "#PWR?" H 8200 5050 50  0001 C CNN
 F 1 "GND" H 8205 5127 50  0000 C CNN
 F 2 "" H 8200 5300 50  0001 C CNN
@@
 	8800 2800 9350 2800
 $Comp
-L power:GND #PWR02
+L power:GND #PWR?
 U 1 1 5F958154
 P 1100 1800
-F 0 "#PWR02" H 1100 1550 50  0001 C CNN
+F 0 "#PWR?" H 1100 1550 50  0001 C CNN
 F 1 "GND" H 1105 1627 50  0000 C CNN
 F 2 "" H 1100 1800 50  0001 C CNN
@@
 $EndComp
 $Comp
-L Device:C C2
+L Device:C C?
 U 1 1 5F9586F2
 P 1500 1600
-F 0 "C2" V 1752 1600 50  0000 C CNN
+F 0 "C?" V 1752 1600 50  0000 C CNN
 F 1 "0.1uF" V 1661 1600 50  0000 C CNN
 F 2 "Capacitor_SMD:C_1206_3216Metric" H 1538 1450 50  0001 C CNN
@@
 	1100 1600 1100 1800
 $Comp
-L Switch:SW_Push SW1
+L Switch:SW_Push SW?
 U 1 1 5F9596F6
 P 1500 1200
-F 0 "SW1" H 1500 1485 50  0000 C CNN
+F 0 "SW?" H 1500 1485 50  0000 C CNN
 F 1 "BOOT" H 1500 1394 50  0000 C CNN
 F 2 "Button_Switch_SMD:SW_SPST_PTS645" H 1500 1400 50  0001 C CNN
@@
 Connection ~ 1900 1200
 $Comp
-L power:GND #PWR05
+L power:GND #PWR?
 U 1 1 5F960D2F
 P 2650 1800
-F 0 "#PWR05" H 2650 1550 50  0001 C CNN
+F 0 "#PWR?" H 2650 1550 50  0001 C CNN
 F 1 "GND" H 2655 1627 50  0000 C CNN
 F 2 "" H 2650 1800 50  0001 C CNN
@@
 $EndComp
 $Comp
-L Device:C C3
+L Device:C C?
 U 1 1 5F960D36
 P 3050 1600
-F 0 "C3" V 3302 1600 50  0000 C CNN
+F 0 "C?" V 3302 1600 50  0000 C CNN
 F 1 "0.1uF" V 3211 1600 50  0000 C CNN
 F 2 "Capacitor_SMD:C_1206_3216Metric" H 3088 1450 50  0001 C CNN
@@
 	2650 1600 2650 1800
 $Comp
-L Switch:SW_Push SW2
+L Switch:SW_Push SW?
 U 1 1 5F960D3E
 P 3050 1200
-F 0 "SW2" H 3050 1485 50  0000 C CNN
+F 0 "SW?" H 3050 1485 50  0000 C CNN
 F 1 "RESET" H 3050 1394 50  0000 C CNN
 F 2 "Button_Switch_SMD:SW_SPST_PTS645" H 3050 1400 50  0001 C CNN
@@
 TXD0
 $Comp
-L Connector_Generic:Conn_02x04_Odd_Even J5
+L Connector_Generic:Conn_02x04_Odd_Even J?
 U 1 1 5FC4BA04
 P 1650 4500
-F 0 "J5" H 1700 4817 50  0000 C CNN
+F 0 "J?" H 1700 4817 50  0000 C CNN
 F 1 "Conn_02x04_Odd_Even" H 1700 4726 50  0000 C CNN
 F 2 "Connector_PinHeader_2.54mm:PinHeader_2x04_P2.54mm_Vertical" H 1650 4500 50  0001 C CNN

Commit message: Reanotate everything and assign missing footprints
Parts:
- gave numbers to parts that had none: 10
Changed lines of the file:
@@
 $EndDescr
 $Comp
-L RF_Module:ESP32-WROOM-32 U?
+L RF_Module:ESP32-WROOM-32 U3
 U 1 1 5F93B762
 P 8200 3700
-F 0 "U?" H 7750 5050 50  0000 C CNN
+F 0 "U3" H 7750 5050 50  0000 C CNN
 F 1 "ESP32-WROOM-32" H 8600 5050 50  0000 C CNN
 F 2 "RF_Module:ESP32-WROOM-32" H 8200 2200 50  0001 C CNN
@@
 $EndComp
 $Comp
-L power:+3V3 #PWR?
+L power:+3V3 #PWR02
 U 1 1 5F9419AA
 P 1100 2650
-F 0 "#PWR?" H 1100 2500 50  0001 C CNN
+F 0 "#PWR02" H 1100 2500 50  0001 C CNN
 F 1 "+3V3" H 1115 2823 50  0000 C CNN
 F 2 "" H 1100 2650 50  0001 C CNN
@@
 $EndComp
 $Comp
-L Device:R R?
+L Device:R R3
 U 1 1 5F94208F
 P 1100 2900
-F 0 "R?" H 1170 2946 50  0000 L CNN
+F 0 "R3" H 1170 2946 50  0000 L CNN
 F 1 "10kR" H 1170 2855 50  0000 L CNN
 F 2 "Resistor_SMD:R_1206_3216Metric" V 1030 2900 50  0001 C CNN
@@
 $EndComp
 $Comp
-L Device:C C?
+L Device:C C1
 U 1 1 5F9429EB
 P 1100 3300
-F 0 "C?" H 1215 3346 50  0000 L CNN
+F 0 "C1" H 1215 3346 50  0000 L CNN
 F 1 "0.1uF" H 1215 3255 50  0000 L CNN
 F 2 "Capacitor_SMD:C_1206_3216Metric" H 1138 3150 50  0001 C CNN
@@
 $EndComp
 $Comp
-L power:GND #PWR?
+L power:GND #PWR03
 U 1 1 5F942C61
 P 1100 3550
-F 0 "#PWR?" H 1100 3300 50  0001 C CNN
+F 0 "#PWR03" H 1100 3300 50  0001 C CNN
 F 1 "GND" H 1105 3377 50  0000 C CNN
 F 2 "" H 1100 3550 50  0001 C CNN
@@
 	1100 2750 1100 2650
 $Comp
-L power:+3V3 #PWR?
+L power:+3V3 #PWR05
 U 1 1 5F943FB0
 P 7350 1600
-F 0 "#PWR?" H 7350 1450 50  0001 C CNN
+F 0 "#PWR05" H 7350 1450 50  0001 C CNN
 F 1 "+3V3" H 7365 1773 50  0000 C CNN
 F 2 "" H 7350 1600 50  0001 C CNN
@@
 $EndComp
 $Comp
-L Device:C C?
+L Device:C C5
 U 1 1 5F9451F0
 P 7800 1850
-F 0 "C?" H 7915 1896 50  0000 L CNN
+F 0 "C5" H 7915 1896 50  0000 L CNN
 F 1 "0.1uF" H 7915 1805 50  0000 L CNN
 F 2 "Capacitor_SMD:C_1206_3216Metric" H 7838 1700 50  0001 C CNN
@@
 $EndComp
 $Comp
-L Device:C C?
+L Device:C C4
 U 1 1 5F946123
 P 7350 1850
-F 0 "C?" H 7465 1896 50  0000 L CNN
+F 0 "C4" H 7465 1896 50  0000 L CNN
 F 1 "22uF" H 7465 1805 50  0000 L CNN
 F 2 "Capacitor_SMD:C_1206_3216Metric" H 7388 1700 50  0001 C CNN
@@
 	7350 2050 7350 2000
 $Comp
-L power:GND #PWR?
+L power:GND #PWR06
 U 1 1 5F947B11
 P 7350 2100
-F 0 "#PWR?" H 7350 1850 50  0001 C CNN
+F 0 "#PWR06" H 7350 1850 50  0001 C CNN
 F 1 "GND" H 7355 1927 50  0000 C CNN
 F 2 "" H 7350 2100 50  0001 C CNN
@@
 	8200 2300 8200 1650
 $Comp
-L power:GND #PWR?
+L power:GND #PWR07
 U 1 1 5F95286C
 P 8200 5300
-F 0 "#PWR?" H 8200 5050 50  0001 C CNN
+F 0 "#PWR07" H 8200 5050 50  0001 C CNN
 F 1 "GND" H 8205 5127 50  0000 C CNN
 F 2 "" H 8200 5300 50  0001 C CNN
@@
 	8800 2800 9350 2800
 $Comp
-L power:GND #PWR?
+L power:GND #PWR01
 U 1 1 5F958154
 P 1100 1800
-F 0 "#PWR?" H 1100 1550 50  0001 C CNN
+F 0 "#PWR01" H 1100 1550 50  0001 C CNN
 F 1 "GND" H 1105 1627 50  0000 C CNN
 F 2 "" H 1100 1800 50  0001 C CNN
@@
 $EndComp
 $Comp
-L Device:C C?
+L Device:C C2
 U 1 1 5F9586F2
 P 1500 1600
-F 0 "C?" V 1752 1600 50  0000 C CNN
+F 0 "C2" V 1752 1600 50  0000 C CNN
 F 1 "0.1uF" V 1661 1600 50  0000 C CNN
 F 2 "Capacitor_SMD:C_1206_3216Metric" H 1538 1450 50  0001 C CNN
@@
 	1100 1600 1100 1800
 $Comp
-L Switch:SW_Push SW?
+L Switch:SW_Push SW2
 U 1 1 5F9596F6
 P 1500 1200
-F 0 "SW?" H 1500 1485 50  0000 C CNN
+F 0 "SW2" H 1500 1485 50  0000 C CNN
 F 1 "BOOT" H 1500 1394 50  0000 C CNN
 F 2 "Button_Switch_SMD:SW_SPST_PTS645" H 1500 1400 50  0001 C CNN
@@
 Connection ~ 1900 1200
 $Comp
-L power:GND #PWR?
+L power:GND #PWR04
 U 1 1 5F960D2F
 P 2650 1800
-F 0 "#PWR?" H 2650 1550 50  0001 C CNN
+F 0 "#PWR04" H 2650 1550 50  0001 C CNN
 F 1 "GND" H 2655 1627 50  0000 C CNN
 F 2 "" H 2650 1800 50  0001 C CNN
@@
 $EndComp
 $Comp
-L Device:C C?
+L Device:C C3
 U 1 1 5F960D36
 P 3050 1600
-F 0 "C?" V 3302 1600 50  0000 C CNN
+F 0 "C3" V 3302 1600 50  0000 C CNN
 F 1 "0.1uF" V 3211 1600 50  0000 C CNN
 F 2 "Capacitor_SMD:C_1206_3216Metric" H 3088 1450 50  0001 C CNN
@@
 	2650 1600 2650 1800
 $Comp
-L Switch:SW_Push SW?
+L Switch:SW_Push SW3
 U 1 1 5F960D3E
 P 3050 1200
-F 0 "SW?" H 3050 1485 50  0000 C CNN
+F 0 "SW3" H 3050 1485 50  0000 C CNN
 F 1 "RESET" H 3050 1394 50  0000 C CNN
 F 2 "Button_Switch_SMD:SW_SPST_PTS645" H 3050 1400 50  0001 C CNN
@@
 TXD0
 $Comp
-L Connector_Generic:Conn_02x04_Odd_Even J?
+L Connector_Generic:Conn_02x04_Odd_Even J5
 U 1 1 5FC4BA04
 P 1650 4500
-F 0 "J?" H 1700 4817 50  0000 C CNN
+F 0 "J5" H 1700 4817 50  0000 C CNN
 F 1 "Conn_02x04_Odd_Even" H 1700 4726 50  0000 C CNN
 F 2 "Connector_PinHeader_2.54mm:PinHeader_2x04_P2.54mm_Vertical" H 1650 4500 50  0001 C CNN
